Commit message: model changes, no movement :boom:
and small eigen fix

File: src/cepheus_description/urdf/cepheus.xacro (robot description, xacro)
@@ -12,5 +12,6 @@
 		</joint> -->
 	</link>
-	<joint name="world_joint" type="continuous">
+	<!-- extra links addition START -->
+	<!-- <joint name="world_joint" type="continuous">
 		<axis xyz="0 0 1"/>
 		<parent link="world"/>
@@ -18,5 +19,96 @@
 		<child link="cepheus"/>
 		<dynamics damping="0" friction="0"/>
-	</joint>
+	</joint> -->
+	<joint name="p1_joint" type="prismatic">
+		<parent link="world"/>
+		<child link="p1"/>
+		<axis xyz="1 0 0"/>
+		<limit lower="-100" upper="100" effort="1000" velocity="10000"/>
+		<dynamics damping="0" friction="0"/>
+	</joint>
+	<link name="p1">
+		<inertial>
+			<origin
+				xyz="0.0 0.0 0.0"
+				rpy="0.0 0.0 0.0" />
+			<mass
+				value="0.01" />
+			<inertia
+				ixx="1e-2"
+				ixy="0.0"
+				ixz="0.0"
+				iyy="1e-2"
+				iyz="0.0"
+				izz="1e-2" />
+		</inertial>
+	</link>
+	<gazebo reference="p1">
+		<mu1>0</mu1>
+		<mu2>0</mu2>
+	</gazebo>
+	<transmission name="lin1">
+		<type>transmission_interface/SimpleTransmission</type>
+		<joint name="p1_joint">
+			<hardwareInterface>hardware_interface/EffortJointInterface</hardwareInterface>
+		</joint>
+		<actuator name="lin_motor1">
+			<hardwareInterface>EffortJointInterface</hardwareInterface>
+			<mechanicalReduction>1</mechanicalReduction>
+		</actuator>
+	</transmission>
+	<joint name="p2_joint" type="prismatic">
+		<parent link="p1"/>
+		<child link="p2"/>
+		<axis xyz="0 1 0"/>
+		<limit lower="-100" upper="100" effort="1000" velocity="10000"/>
+		<dynamics damping="0" friction="0"/>
+	</joint>
+	<link name="p2">
+		<inertial>
+			<origin
+				xyz="0.0 0.0 0.0"
+				rpy="0.0 0.0 0.0" />
+			<mass
+				value="0.01" />
+			<inertia
+				ixx="1e-2"
+				ixy="0.0"
+				ixz="0.0"
+				iyy="1e-2"
+				iyz="0.0"
+				izz="1e-2" />
+		</inertial>
+		<surface>
+			<friction>
+				<ode>
+					<mu>0</mu>
+					<mu2>0</mu2>
+					<fdir1>0 1.0 0</fdir1>
+					<implicit_spring_damper>true</implicit_spring_damper>
+				</ode>
+			</friction>
+		</surface>
+	</link>
+	<gazebo reference="p2">
+		<mu1>0</mu1>
+		<mu2>0</mu2>
+	</gazebo>
+	<transmission name="lin2">
+		<type>transmission_interface/SimpleTransmission</type>
+		<joint name="p2_joint">
+			<hardwareInterface>hardware_interface/EffortJointInterface</hardwareInterface>
+		</joint>
+		<actuator name="lin_motor2">
+			<hardwareInterface>EffortJointInterface</hardwareInterface>
+			<mechanicalReduction>1</mechanicalReduction>
+		</actuator>
+	</transmission>
+	<joint name="r_joint" type="continuous">
+		<axis xyz="0 0 1"/>
+		<parent link="p2"/>
+		<origin rpy="0 0 0" xyz="0 0 0"/>
+		<child link="cepheus"/>
+	</joint>
+	<!-- extra links addition END -->
 	<link name="cepheus">
 		<inertial>
@@ -85,6 +177,5 @@
 			transmission_interface/SimpleTransmission</type>
 		<joint name="reaction_wheel_joint">
-			<hardwareInterface>
-			EffortJointInterface</hardwareInterface>
+			<hardwareInterface>hardware_interface/EffortJointInterface</hardwareInterface>
 		</joint>
 		<actuator name="motor1">
@@ -155,6 +246,5 @@
 			transmission_interface/SimpleTransmission</type>
 		<joint name="left_shoulder">
-			<hardwareInterface>
-			EffortJointInterface</hardwareInterface>
+			<hardwareInterface>hardware_interface/EffortJointInterface</hardwareInterface>
 		</joint>
 		<actuator name="motor2">
@@ -225,6 +315,5 @@
 			transmission_interface/SimpleTransmission</type>
 		<joint name="left_elbow">
-			<hardwareInterface>
-				EffortJointInterface</hardwareInterface>
+			<hardwareInterface>hardware_interface/EffortJointInterface</hardwareInterface>
 		</joint>
 		<actuator name="motor3">

Commit message: movement fix
add gazebo reference cepheus in xarco

File: src/cepheus_description/urdf/cepheus.xacro (robot description, xacro)
@@ -32,6 +32,5 @@
 				xyz="0.0 0.0 0.0"
 				rpy="0.0 0.0 0.0" />
-			<mass
-				value="0.01" />
+			<mass value="0.01" />
 			<inertia
 				ixx="1e-2"
@@ -61,6 +60,12 @@
 		<child link="p2"/>
 		<axis xyz="0 1 0"/>
-		<limit lower="-100" upper="100" effort="1000" velocity="10000"/>
-		<dynamics damping="0" friction="0"/>
+		<limit
+			lower="-100"
+			upper="100"
+			effort="1000"
+			velocity="10000"/>
+		<dynamics
+			damping="0"
+			friction="0"/>
 	</joint>
 	<link name="p2">
@@ -69,6 +74,5 @@
 				xyz="0.0 0.0 0.0"
 				rpy="0.0 0.0 0.0" />
-			<mass
-				value="0.01" />
+			<mass value="0.01" />
 			<inertia
 				ixx="1e-2"
@@ -114,22 +118,21 @@
 		<inertial>
 			<origin
-			xyz="0.0024 0.02937 0.15711"
-			rpy="0 0 0" />
-			<mass
-			value="7.11891369052411" />
-			<inertia
-			ixx="0.0937165866660239"
-			ixy="-0.004838152027527" ixz="-0.00397891305009112"
-			iyy="0.0905199286322999"
-			iyz="-0.00257712868335304"
-			izz="0.0755866683160163" />
-		</inertial>
-		<visual>
-			<origin
-			xyz="0 0 0"
-			rpy="0 0 0" />
-			<geometry>
-				<mesh
-				filename="package://cepheus_description/urdf/meshes/cepheus.STL" />
+				xyz="0.0024 0.02937 0.15711"
+				rpy="0 0 0" />
+			<mass value="7.11891369052411" />
+			<inertia
+				ixx="0.0937165866660239"
+				ixy="-0.004838152027527"
+				ixz="-0.00397891305009112"
+				iyy="0.0905199286322999"
+				iyz="-0.00257712868335304"
+				izz="0.0755866683160163" />
+		</inertial>
+		<visual>
+			<origin
+				xyz="0 0 0"
+				rpy="0 0 0" />
+			<geometry>
+				<mesh filename="package://cepheus_description/urdf/meshes/cepheus.STL" />
 			</geometry>
 			<material name="LightGrey"/>
@@ -137,6 +140,6 @@
 		<collision>
 			<origin
-			xyz="0 0 0.215"
-			rpy="0 0 0" />
+				xyz="0 0 0.215"
+				rpy="0 0 0" />
 			<geometry>
 				<cylinder length="0.43" radius="0.2"/>
@@ -156,6 +159,5 @@
 			</material>
 			<geometry>
-				<mesh
-				filename="package://cepheus_description/urdf/meshes/reaction_wheel.STL" />
+				<mesh filename="package://cepheus_description/urdf/meshes/reaction_wheel.STL" />
 			</geometry>
 			<origin xyz="0 0 0" rpy="0 0 0"/>
@@ -173,4 +175,8 @@
 		</inertial>
 	</link>
+	<gazebo reference="cepheus">
+		<mu1>0</mu1>
+		<mu2>0</mu2>
+	</gazebo>
 	<transmission name="tran1">
 		<type>
@@ -180,39 +186,30 @@
 		</joint>
 		<actuator name="motor1">
-			<hardwareInterface>
-				EffortJointInterface</hardwareInterface>
-			<mechanicalReduction>
-				1</mechanicalReduction>
-		</actuator>
-	</transmission>
-	<joint
-		name="left_shoulder"
-		type="revolute">
+			<hardwareInterface>EffortJointInterface</hardwareInterface>
+			<mechanicalReduction>1</mechanicalReduction>
+		</actuator>
+	</transmission>
+	<joint name="left_shoulder" type="revolute">
 		<origin
-		xyz="0.17271 0.091404 0.05875"
-		rpy="0 0 0" />
-		<parent
-		link="cepheus" />
-		<child
-		link="left_arm" />
-		<axis
-		xyz="0 0 1" />
+			xyz="0.17271 0.091404 0.05875"
+			rpy="0 0 0" />
+		<parent link="cepheus" />
+		<child link="left_arm" />
+		<axis xyz="0 0 1" />
 		<limit
-		lower="-0.86"
-		upper="2.54"
-		effort="20"
-		velocity="20" />
+			lower="-0.86"
+			upper="2.54"
+			effort="20"
+			velocity="20" />
 		<dynamics
-		damping="1"
-		friction="1" />
-	</joint>
-	<link
-		name="left_arm">
+			damping="1"
+			friction="1" />
+	</joint>
+	<link name="left_arm">
 		<inertial>
 			<origin
 				xyz="0.10516 0.00268 0.00996"
 				rpy="0 0 0" />
-			<mass
-				value="0.07974" />
+			<mass value="0.07974" />
 			<inertia
 				ixx="0.0971318625270812"
@@ -228,6 +225,5 @@
 				rpy="0 0 0" />
 			<geometry>
-				<mesh
-					filename="package://cepheus_description/urdf/meshes/left_arm.STL" />
+				<mesh filename="package://cepheus_description/urdf/meshes/left_arm.STL" />
 			</geometry>
 			<material name="LightGrey"/>
@@ -243,28 +239,20 @@
 	</link>
 	<transmission name="tran2">
-		<type>
-			transmission_interface/SimpleTransmission</type>
+		<type>transmission_interface/SimpleTransmission</type>
 		<joint name="left_shoulder">
 			<hardwareInterface>hardware_interface/EffortJointInterface</hardwareInterface>
 		</joint>
 		<actuator name="motor2">
-			<hardwareInterface>
-				EffortJointInterface</hardwareInterface>
-			<mechanicalReduction>
-				1</mechanicalReduction>
-		</actuator>
-	</transmission>
-	<joint
-		name="left_elbow"
-		type="revolute">
+			<hardwareInterface>EffortJointInterface</hardwareInterface>
+			<mechanicalReduction>1</mechanicalReduction>
+		</actuator>
+	</transmission>
+	<joint name="left_elbow" type="revolute">
 		<origin
 			xyz="0.18120 -0.01176 -0.002"
 			rpy="0 0 0" />
-		<parent
-			link="left_arm" />
-		<child
-			link="left_forearm" />
-		<axis
-			xyz="0 0 1" />
+		<parent link="left_arm" />
+		<child link="left_forearm" />
+		<axis xyz="0 0 1" />
 		<limit
 			lower="-3.14"
@@ -276,12 +264,10 @@
 			friction="1" />
 	</joint>
-	<link
-		name="left_forearm">
+	<link name="left_forearm">
 		<inertial>
 			<origin
 				xyz="0.06831 0.00878 0.01558"
 				rpy="0 0 0" />
-			<mass
-				value="0.06392" />
+			<mass value="0.06392" />
 			<inertia
 				ixx="1"
@@ -297,6 +283,5 @@
 				rpy="0 0 0" />
 			<geometry>
-				<mesh
-					filename="package://cepheus_description/urdf/meshes/left_forearm.STL" />
+				<mesh filename="package://cepheus_description/urdf/meshes/left_forearm.STL" />
 			</geometry>
 			<material name="LightGrey"/>
@@ -304,6 +289,6 @@
 		<collision>
 			<origin
-			xyz="0.105 0.0115 0.0125"
-			rpy="0 0 0" />
+				xyz="0.105 0.0115 0.0125"
+				rpy="0 0 0" />
 			<geometry>
 				<box size="0.13 0.025 0.025"/>
@@ -312,28 +297,20 @@
 	</link>
 	<transmission name="tran3">
-		<type>
-			transmission_interface/SimpleTransmission</type>
+		<type>transmission_interface/SimpleTransmission</type>
 		<joint name="left_elbow">
 			<hardwareInterface>hardware_interface/EffortJointInterface</hardwareInterface>
 		</joint>
 		<actuator name="motor3">
-			<hardwareInterface>
-				EffortJointInterface</hardwareInterface>
-			<mechanicalReduction>
-				1</mechanicalReduction>
-		</actuator>
-	</transmission>
-	<joint
-		name="left_wrist"
-		type="fixed">
+			<hardwareInterface>EffortJointInterface</hardwareInterface>
+			<mechanicalReduction>1</mechanicalReduction>
+		</actuator>
+	</transmission>
+	<joint name="left_wrist" type="fixed">
 		<origin
 			xyz="0.15965 0.01176 -0.00838"
 			rpy="0 0 0 " />
-		<parent
-			link="left_forearm" />
-		<child
-			link="left_grip" />
-		<axis
-			xyz="0 0 1" />
+		<parent link="left_forearm" />
+		<child link="left_grip" />
+		<axis xyz="0 0 1" />
 		<limit
 			lower="-1.570796327"
@@ -345,12 +322,10 @@
 			friction="1" />
 	</joint>
-	<link
-		name="left_grip">
+	<link name="left_grip">
 		<inertial>
 			<origin
 				xyz="0.01947 -0.00226 -0.00228"
 				rpy="0 0 0" />
-			<mass
-				value="0.03547" />
+			<mass value="0.03547" />
 			<inertia
 				ixx="0.0926325136613974"

Commit message: mount camera
old upds in values

File: src/cepheus_description/urdf/cepheus.xacro (robot description, xacro)
@@ -3,4 +3,5 @@
 	<xacro:include filename="$(find cepheus_description)/urdf/cepheus.gazebo" />
 	<xacro:include filename="$(find cepheus_description)/urdf/materials.xacro" />
+	<xacro:property name="camera_link" value="0.05" /> <!-- Size of square 'camera' box -->
 	<link name="world">
 		<!-- <joint name="world_joint" type="continuous">
@@ -120,12 +121,12 @@
 				xyz="0.0024 0.02937 0.15711"
 				rpy="0 0 0" />
-			<mass value="7.11891369052411" />
-			<inertia
-				ixx="0.0937165866660239"
-				ixy="-0.004838152027527"
-				ixz="-0.00397891305009112"
-				iyy="0.0905199286322999"
-				iyz="-0.00257712868335304"
-				izz="0.0755866683160163" />
+			<mass value="13.3" />
+			<inertia
+				ixx="0"
+				ixy="0"
+				ixz="0"
+				iyy="0"
+				iyz="0"
+				izz="0.160875" />
 		</inertial>
 		<visual>
@@ -209,14 +210,14 @@
 		<inertial>
 			<origin
-				xyz="0.10516 0.00268 0.00996"
-				rpy="0 0 0" />
-			<mass value="0.07974" />
-			<inertia
-				ixx="0.0971318625270812"
-				ixy="0.00469370636895255"
-				ixz="-0.000908920687249813"
-				iyy="0.0755866683160163"
-				iyz="0.000665178045940108"
-				izz="0.0871046527712426" />
+				xyz="0.119 0 0"
+				rpy="0 0 0" />
+			<mass value="0.083" />
+			<inertia
+				ixx="0"
+				ixy="0"
+				ixz="0"
+				iyy="0"
+				iyz="0"
+				izz="0.000346" />
 		</inertial>
 		<visual>
@@ -250,5 +251,5 @@
 	<joint name="left_elbow" type="revolute">
 		<origin
-			xyz="0.18120 -0.01176 -0.002"
+			xyz="0.1810 0 0"
 			rpy="0 0 0" />
 		<parent link="left_arm" />
@@ -267,14 +268,14 @@
 		<inertial>
 			<origin
-				xyz="0.06831 0.00878 0.01558"
-				rpy="0 0 0" />
-			<mass value="0.06392" />
-			<inertia
-				ixx="1"
-				ixy="1"
-				ixz="1"
-				iyy="1"
-				iyz="1"
-				izz="1" />
+				xyz="0.119 0 0"
+				rpy="0 0 0" />
+			<mass value="0.187" />
+			<inertia
+				ixx="0"
+				ixy="0"
+				ixz="0"
+				iyy="0"
+				iyz="0"
+				izz="0.000346" />
 		</inertial>
 		<visual>
@@ -305,5 +306,5 @@
 			<mechanicalReduction>1</mechanicalReduction>
 		</actuator>
-	</transmission>
+	</transmission><!--
 	<joint name="left_wrist" type="fixed">
 		<origin
@@ -353,4 +354,31 @@
 			</geometry>
 		</collision>
+	</link> -->
+	<joint name="camera_joint" type="fixed">
+		<axis xyz="0 1 0" />
+		<origin xyz="0 0 3.0" rpy="0 0 0"/>
+		<parent link="world"/>
+		<child link="camera_link"/>
+	</joint>
+	<!-- Camera -->
+	<link name="camera_link">
+		<collision>
+			<origin xyz="0 0 0" rpy="0 0 0"/>
+			<geometry>
+				<box size="${camera_link} ${camera_link} ${camera_link}"/>
+			</geometry>
+		</collision>
+		<visual>
+			<origin xyz="0 0 0" rpy="0 0 0"/>
+			<geometry>
+				<box size="${camera_link} ${camera_link} ${camera_link}"/>
+			</geometry>
+			<material name="red"/>
+		</visual>
+		<inertial>
+			<mass value="1e-5" />
+			<origin xyz="0 0 0" rpy="0 0 0"/>
+			<inertia ixx="1e-6" ixy="0" ixz="0" iyy="1e-6" iyz="0" izz="1e-6" />
+		</inertial>
 	</link>
 </robot>

Commit message: stream gazebo top down camera to react

File: src/cepheus_description/urdf/cepheus.xacro (robot description, xacro)
@@ -357,5 +357,5 @@
 	<joint name="camera_joint" type="fixed">
 		<axis xyz="0 1 0" />
-		<origin xyz="0 0 3.0" rpy="0 0 0"/>
+		<origin xyz="0 0 3.0" rpy="0 1.5708 1.5708"/>
 		<parent link="world"/>
 		<child link="camera_link"/>
